File: hardware/PCB/STIC.kicad_sch (KiCad schematic)
At the start: 26 parts, among them J1 22-03-5035, J2 53047-0510, J3 53047-0310, J4 3 way molex cable, J5 Conn_01x02, U1 XIAO_BLE, U2 RM3100_Breakout, U3 OLED1_3_GND1, U4 XIAO_RM3100_Breakout

Commit message: Get files ready for SMT production
Parts:
- BT1, J1, J2, J3, J4, J5, LASER1, U1, U2, U3, U4: now not fitted
- CHARGER1: value XC6802A42XMR-G -> XC6802A42XPR-G
- C_1: renamed from C1; now not fitted
- C_2: renamed from C2; now not fitted
- C_3: renamed from C3; now not fitted
- R_1: renamed from R1; now not fitted
- R_2: renamed from R2; now not fitted
- R_3: renamed from R3; now not fitted
- renumbered C1a1 to C1, C2a1 to C2, C3a1 to C3, R1a1 to R1, R2a1 to R2, R3a1 to R3
